File: kicad/binClock/binClock.kicad_pcb (KiCad board)
At the start: 2 copper layers, 93 x 59.5 mm, 56 parts, among them M2.5 MountingHole_Pad, SW1 SW_Push, SW2 SW_Push

Commit message: Corrected error in schematic and recreated production files
Parts:
- removed REF**: OSHW-Logo2_14.6x12mm_SilkScreen, Symbol:OSHW-Logo2_14.6x12mm_SilkScreen
- C1, C2, C3, C4: value C_Small -> 100n
- H5, H6: renamed from LED GND
- R1, R11, R12, R13, R14, R17, R18, R19, R2, R20, R21, R22, R25, R26, R27, R28, R29, R3, R30, R33, R34, R4, R7, R8: value R -> 200
- R10, R9: value R -> 10k
- R15, R16, R23, R24, R31, R32, R5, R6: value R -> 510
- U1: renamed from Register 4; value ~ -> 74HC595N
- U2: renamed from Register 3; value ~ -> 74HC595N
- U3: renamed from ESP32-C3 Supermini
- U4: renamed from Register 2; value ~ -> 74HC595N
- U5: renamed from Register 1; value ~ -> 74HC595N
- renumbered M2.5 to H1, M2.5 to H2, M2.5 to H3, M2.5 to H4, R4 to J1, R3 to J2, R2 to J3, R1 to J4
Connections:
- U2 pad 14: Net-(U1-SER) -> Net-(U2-SER)
- U2 pad 9: unconnected-(U2-QH*-Pad9) -> Net-(U1-SER)
- U4 pad 9: Net-(U1-SER) -> Net-(U2-SER)
Routing:
- net Net-(U1-SER): track 61.4 -> 10.2 mm, vias 2 -> 0
- net Net-(U2-SER): track 0.00 -> 25.8 mm, vias 0 -> 2
- net GND: vias 3 -> 4
Other:
- board text added: "binClock v1.0.1 Daniel Colon helder.uk"
- board text removed: "binClock v1.0.0 Daniel Colon helder.uk"
